File: Pike/Pike.kicad_pcb (KiCad board)
At the start: 2 copper layers, 87.5 x 27.1 mm, 19 parts, among them J1 PJ-005A, J2 Power bus 02x08

Commit message: all gathered
Parts:
- D1, D3, D4: value IR204A -> 604-WP424GDT
