File: Pike/Pike.kicad_sch (KiCad schematic)
At the start: 19 parts, among them J1 PJ-005A, J2 Power bus 02x08

Commit message: all gathered
Parts:
- C1, C2: Comments (none) -> Low height (7mm); Mouser Part Number (none) -> 667-ECE-A1HKA220
- D1, D3, D4: Comments (none) -> You can adjust LEDs and corresponding resistors on your own; Mouser Part Number (none) -> 604-WP424GDT
- D2: Mouser Part Number (none) -> 863-1N5400G
- J1: Mouser Part Number (none) -> 490-PJ-005A
- PS2: Comments (none) -> 495-TSR-1-2450 is also OK
- R1, R2: Mouser Part Number (none) -> CFR25SJT-26-2K2
- R3: Mouser Part Number (none) -> CFR-25JB-1K0
- TP1: now left out of the parts list
